File: cores/s18/sch/amd.kicad_sch (KiCad schematic)
At the start: 88 parts, among them IC92 TL084, IC93 TL084, IC94 MB3733-31

Commit message: system 18 schematics transferred after update
Parts:
- R60: value AUSENTE -> R
Connections:
- net ?: no longer IC94.6 (AUDIO_MUTE)
Other:
- note added: "NOT MOUNTED"
Changed lines of the file:
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@@
     (stroke (width 0) (type default) (color 0 0 0 0))
   )
-  (wire (pts (xy 41.91 210.82) (xy 34.29 210.82))
+  (wire (pts (xy 41.91 210.82) (xy 35.56 210.82))
     (stroke (width 0) (type default) (color 0 0 0 0))
   )
@@
     (stroke (width 0) (type default) (color 0 0 0 0))
   )
-  (image (at 419.1 262.89) (scale 0.25)
+  (image (at 398.78 260.35) (scale 0.25)
     (data
       iVBORw0KGgoAAAANSUhEUgAAAxoAAAMaCAIAAACOIqcFAAAAA3NCSVQICAjb4U/gAAAACXBIWXMA
@@
     )
   )
+  (text "NOT MOUNTED" (at 223.52 166.37 0)
+    (effects (font (size 1.27 1.27)) (justify left bottom))
+  )
   (text "9v\n" (at 219.71 107.95 0)
     (effects (font (size 1.27 1.27)) (justify left bottom))
@@
     (effects (font (size 1.27 1.27)) (justify left bottom))
   )
-  (label "?" (at 368.3 52.07 270)
-    (effects (font (size 1.27 1.27)) (justify right bottom))
-  )
   (label "VSS" (at 242.57 176.53 180)
     (effects (font (size 1.27 1.27)) (justify right bottom))
@@
     (effects (font (size 1.27 1.27)) (justify right))
   )
-  (hierarchical_label "ASSP_36" (shape input) (at 34.29 210.82 180)
+  (hierarchical_label "ASSP_36" (shape input) (at 35.56 210.82 180)
     (effects (font (size 1.27 1.27)) (justify right))
   )
@@
   (symbol (lib_id "power:VCC") (at 133.35 30.48 0) (unit 1)
     (in_bom yes) (on_board yes)
-    (property "Reference" "#PWR0126" (id 0) (at 133.35 34.29 0)
+    (property "Reference" "#PWR?" (id 0) (at 133.35 34.29 0)
       (effects (font (size 1.27 1.27)) hide)
     )
@@
   (symbol (lib_id "power:VSS") (at 251.46 85.09 180) (unit 1)
     (in_bom yes) (on_board yes)
-    (property "Reference" "#PWR0125" (id 0) (at 251.46 81.28 0)
+    (property "Reference" "#PWR?" (id 0) (at 251.46 81.28 0)
       (effects (font (size 1.27 1.27)) hide)
     )
@@
   (symbol (lib_id "power:VCC") (at 393.7 41.91 0) (unit 1)
     (in_bom yes) (on_board yes)
-    (property "Reference" "#PWR0124" (id 0) (at 393.7 45.72 0)
+    (property "Reference" "#PWR?" (id 0) (at 393.7 45.72 0)
       (effects (font (size 1.27 1.27)) hide)
     )
@@
     (in_bom yes) (on_board yes)
     (property "Reference" "R60" (id 0) (at 245.11 165.1 0))
-    (property "Value" "AUSENTE" (id 1) (at 240.03 168.91 90))
+    (property "Value" "R" (id 1) (at 245.11 168.91 0))
     (property "Footprint" "" (id 2) (at 243.586 169.164 90)
       (effects (font (size 1.27 1.27)) hide)
