File: cores/s18/sch/blanking.kicad_sch (KiCad schematic)
At the start: 26 parts, among them IC66 74HC4066, IC67 74HC4066

Commit message: system 18 schematics transferred after update
Connections:
- net GREEN_A: now also FL24.1, FL24.3, IC66.3 (2Z), IC67.3 (2Z); no longer FL23.1, FL23.3, IC66.2 (1Z), IC67.2 (1Z)
- net RED_A: now also FL23.1, FL23.3, IC66.2 (1Z), IC67.2 (1Z); no longer FL24.1, FL24.3, IC66.3 (2Z), IC67.3 (2Z)
Changed lines of the file:
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@@
     (effects (font (size 1.27 1.27)) (justify right bottom))
   )
-  (label "RED_A" (at 68.58 137.16 180)
+  (label "RED_A" (at 48.26 137.16 180)
     (effects (font (size 1.27 1.27)) (justify right bottom))
   )
-  (label "GREEN_A" (at 48.26 137.16 180)
+  (label "GREEN_A" (at 68.58 137.16 180)
     (effects (font (size 1.27 1.27)) (justify right bottom))
   )
@@
     (effects (font (size 1.27 1.27)) (justify right))
   )
-  (hierarchical_label "GREEN_A" (shape bidirectional) (at 81.28 97.79 180)
+  (hierarchical_label "GREEN_A" (shape bidirectional) (at 77.47 100.33 180)
     (effects (font (size 1.27 1.27)) (justify right))
   )
@@
     (effects (font (size 1.27 1.27)) (justify right))
   )
-  (hierarchical_label "RED_A" (shape bidirectional) (at 77.47 100.33 180)
+  (hierarchical_label "RED_A" (shape bidirectional) (at 81.28 97.79 180)
     (effects (font (size 1.27 1.27)) (justify right))
   )
