File: cores/s18/sch/colmix.kicad_sch (KiCad schematic)
At the start: 7 parts

Commit message: system 18 schematics transferred after update
Connections:
- net A0 renamed COLA0
- net A1 renamed COLA1
- net A10 renamed COLA10
- net A2 renamed COLA2
- net A3 renamed COLA3
- net A4 renamed COLA4
- net A5 renamed COLA5
- net A6 renamed COLA6
- net A7 renamed COLA7
- net A8 renamed COLA8
- net A9 renamed COLA9
- net D0 renamed RGB0
- net D1 renamed RGB1
- net D10 renamed RGB10
- net D11 renamed RGB11
- net D12 renamed RGB12
- net D13 renamed RGB13
- net D14 renamed RGB14
- net D15 renamed RGB15
- net D2 renamed RGB2
- net D3 renamed RGB3
- net D4 renamed RGB4
- net D5 renamed RGB5
- net D6 renamed RGB6
- net D7 renamed RGB7
- net D8 renamed RGB8
- net D9 renamed RGB9
- net HI_LO: no longer names the net of E8.28 (HI/LO)
- net MAIN_A1 renamed MAIN_AB1
- net MAIN_A10 renamed MAIN_AB10
- net MAIN_A11 renamed MAIN_AB11
- net MAIN_A2 renamed MAIN_AB2
- net MAIN_A3 renamed MAIN_AB3
- net MAIN_A4 renamed MAIN_AB4
- net MAIN_A5 renamed MAIN_AB5
- net MAIN_A6 renamed MAIN_AB6
- net MAIN_A7 renamed MAIN_AB7
- net MAIN_A8 renamed MAIN_AB8
- net MAIN_A9 renamed MAIN_AB9
- net MAIN_D0 renamed MAIN_DB0
- net MAIN_D1 renamed MAIN_DB1
- net MAIN_D10 renamed MAIN_DB10
- net MAIN_D11 renamed MAIN_DB11
- net MAIN_D12 renamed MAIN_DB12
- net MAIN_D13 renamed MAIN_DB13
- net MAIN_D14 renamed MAIN_DB14
- net MAIN_D15 renamed MAIN_DB15
- net MAIN_D2 renamed MAIN_DB2
- net MAIN_D3 renamed MAIN_DB3
- net MAIN_D4 renamed MAIN_DB4
- net MAIN_D5 renamed MAIN_DB5
- net MAIN_D6 renamed MAIN_DB6
- net MAIN_D7 renamed MAIN_DB7
- net MAIN_D8 renamed MAIN_DB8
- net MAIN_D9 renamed MAIN_DB9
- net ~{BLANK}: no longer names the net of E8.27 (~{BLANK})
Other:
- note removed: "COLMIX"
