File: cores/s18/sch/cpurom.kicad_sch (KiCad schematic)
At the start: 6 parts

Commit message: system 18 schematics transferred after update
Connections:
- net MAIN_A1 renamed MAIN_AB1
- net MAIN_A10 renamed MAIN_AB10
- net MAIN_A11 renamed MAIN_AB11
- net MAIN_A12 renamed MAIN_AB12
- net MAIN_A13 renamed MAIN_AB13
- net MAIN_A14 renamed MAIN_AB14
- net MAIN_A15 renamed MAIN_AB15
- net MAIN_A16 renamed MAIN_AB16
- net MAIN_A17 renamed MAIN_AB17
- net MAIN_A18 renamed MAIN_AB18
- net MAIN_A2 renamed MAIN_AB2
- net MAIN_A3 renamed MAIN_AB3
- net MAIN_A4 renamed MAIN_AB4
- net MAIN_A5 renamed MAIN_AB5
- net MAIN_A6 renamed MAIN_AB6
- net MAIN_A7 renamed MAIN_AB7
- net MAIN_A8 renamed MAIN_AB8
- net MAIN_A9 renamed MAIN_AB9
- net MAIN_D0 renamed MAIN_DB0
- net MAIN_D1 renamed MAIN_DB1
- net MAIN_D10 renamed MAIN_DB10
- net MAIN_D11 renamed MAIN_DB11
- net MAIN_D12 renamed MAIN_DB12
- net MAIN_D13 renamed MAIN_DB13
- net MAIN_D14 renamed MAIN_DB14
- net MAIN_D15 renamed MAIN_DB15
- net MAIN_D2 renamed MAIN_DB2
- net MAIN_D3 renamed MAIN_DB3
- net MAIN_D4 renamed MAIN_DB4
- net MAIN_D5 renamed MAIN_DB5
- net MAIN_D6 renamed MAIN_DB6
- net MAIN_D7 renamed MAIN_DB7
- net MAIN_D8 renamed MAIN_DB8
- net MAIN_D9 renamed MAIN_DB9
