File: cores/s18/sch/gfx_main.kicad_sch (KiCad schematic)
At the start: 15 parts, among them IC69 MB8461-12, IC70 MB8461-12

Commit message: system 18 schematics transferred after update
Connections:
- net at V10.104 (~{IPL1}): no longer V10.105 (~{IPL2})
- net ~{CSYNC}: now reaches V10.42 (~{CSYNC})
- net ~{CSYNC}: no longer V10.41 (~{VSYNC})
- net at V10.50 (SBCR): no longer V10.51 (CLK0)
- net A0 renamed BDP0
- net A1 renamed BDP1
- net A2 renamed BDP2
- net A3 renamed BDP3
- net A4 renamed BDP4
- net A5 renamed BDP5
- net A6 renamed BDP6
- net A7 renamed BDP7
- net MAIN_A1 renamed MAIN_AB1
- net MAIN_A10 renamed MAIN_AB10
- net MAIN_A11 renamed MAIN_AB11
- net MAIN_A12 renamed MAIN_AB12
- net MAIN_A13 renamed MAIN_AB13
- net MAIN_A14 renamed MAIN_AB14
- net MAIN_A15 renamed MAIN_AB15
- net MAIN_A16 renamed MAIN_AB16
- net MAIN_A17 renamed MAIN_AB17
- net MAIN_A18 renamed MAIN_AB18
- net MAIN_A19 renamed MAIN_AB19
- net MAIN_A2 renamed MAIN_AB2
- net MAIN_A20 renamed MAIN_AB20
- net MAIN_A21 renamed MAIN_AB21
- net MAIN_A22 renamed MAIN_AB22
- net MAIN_A23 renamed MAIN_AB23
- net MAIN_A3 renamed MAIN_AB3
- net MAIN_A4 renamed MAIN_AB4
- net MAIN_A5 renamed MAIN_AB5
- net MAIN_A6 renamed MAIN_AB6
- net MAIN_A7 renamed MAIN_AB7
- net MAIN_A8 renamed MAIN_AB8
- net MAIN_A9 renamed MAIN_AB9
- net MAIN_D0 renamed MAIN_DB0
- net MAIN_D1 renamed MAIN_DB1
- net MAIN_D10 renamed MAIN_DB10
- net MAIN_D11 renamed MAIN_DB11
- net MAIN_D12 renamed MAIN_DB12
- net MAIN_D13 renamed MAIN_DB13
- net MAIN_D14 renamed MAIN_DB14
- net MAIN_D15 renamed MAIN_DB15
- net MAIN_D2 renamed MAIN_DB2
- net MAIN_D3 renamed MAIN_DB3
- net MAIN_D4 renamed MAIN_DB4
- net MAIN_D5 renamed MAIN_DB5
- net MAIN_D6 renamed MAIN_DB6
- net MAIN_D7 renamed MAIN_DB7
- net MAIN_D8 renamed MAIN_DB8
- net MAIN_D9 renamed MAIN_DB9
- net SEL0: no longer names the net of RA22.2 (R1), V10.45 (SEL0)
- net ~{HL}: no longer names the net of RA22.4 (R3), V10.44 (~{HL})
- net ~{HSYNC}: no longer names the net of RA22.9 (R8), V10.43 (~{HSYNC})
- new net ~{VSYNC}: V10.41 (~{VSYNC})
- now unconnected: V10.100 (~{BGAK}), V10.115 (~{UWR}), V10.116 (~{LWR}), V10.117 (~{OE0}), V10.118 (~{CAS0}), V10.119 (~{RAS0}), V10.120 (RA0), V10.121 (RA1), V10.122 (RA2), V10.123 (RA3), V10.124 (RA4), V10.125 (RA5), V10.126 (RA6), V10.127 (RA7), V10.18 (RD0), V10.19 (RD1), V10.20 (RD2), V10.21 (RD3), V10.22 (RD4), V10.23 (RD5), V10.24 (RD6), V10.25 (RD7), V10.98 (~{INT}), V10.99 (~{BR})
- no-connect marks 15 -> 36
Other:
- note added: "BIT DUAL PORT DYNAMIC RANDOM ACCESS MEMORY"
- note added: "PIN19S11"
- note added: "PIN3R11"
- note removed: "?"
- moved on the sheet: RA21, RA22
