File: cores/s18/sch/gfx_obj.kicad_sch (KiCad schematic)
At the start: 14 parts, among them U8 CY7C128-45PC, X7 74LS245, X8 74LS244, Y7 74LS244, Y8 CY7C128-45PC

Commit message: system 18 schematics transferred after update
Connections:
- net MAIN_A1 renamed MAIN_AB1
- net MAIN_A10 renamed MAIN_AB10
- net MAIN_A2 renamed MAIN_AB2
- net MAIN_A3 renamed MAIN_AB3
- net MAIN_A4 renamed MAIN_AB4
- net MAIN_A5 renamed MAIN_AB5
- net MAIN_A6 renamed MAIN_AB6
- net MAIN_A7 renamed MAIN_AB7
- net MAIN_A8 renamed MAIN_AB8
- net MAIN_A9 renamed MAIN_AB9
- net MAIN_D0 renamed MAIN_DB0
- net MAIN_D1 renamed MAIN_DB1
- net MAIN_D10 renamed MAIN_DB10
- net MAIN_D11 renamed MAIN_DB11
- net MAIN_D12 renamed MAIN_DB12
- net MAIN_D13 renamed MAIN_DB13
- net MAIN_D14 renamed MAIN_DB14
- net MAIN_D15 renamed MAIN_DB15
- net MAIN_D2 renamed MAIN_DB2
- net MAIN_D3 renamed MAIN_DB3
- net MAIN_D4 renamed MAIN_DB4
- net MAIN_D5 renamed MAIN_DB5
- net MAIN_D6 renamed MAIN_DB6
- net MAIN_D7 renamed MAIN_DB7
- net MAIN_D8 renamed MAIN_DB8
- net MAIN_D9 renamed MAIN_DB9
Changed lines of the file:
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@@
     (effects (font (size 1.27 1.27)) (justify right bottom))
   )
-  (label "MAIN_A1" (at 133.35 187.96 90)
-    (effects (font (size 1.27 1.27)) (justify left bottom))
-  )
-  (label "MAIN_D15" (at 275.59 190.5 0)
+  (label "MAIN_AB1" (at 133.35 187.96 90)
+    (effects (font (size 1.27 1.27)) (justify left bottom))
+  )
+  (label "MAIN_DB15" (at 275.59 190.5 0)
     (effects (font (size 1.27 1.27)) (justify left bottom))
   )
@@
     (effects (font (size 1.27 1.27)) (justify right bottom))
   )
-  (label "MAIN_A2" (at 135.89 187.96 90)
+  (label "MAIN_AB2" (at 135.89 187.96 90)
     (effects (font (size 1.27 1.27)) (justify left bottom))
   )
@@
     (effects (font (size 1.27 1.27)) (justify left bottom))
   )
-  (label "MAIN_D11" (at 275.59 200.66 0)
+  (label "MAIN_DB11" (at 275.59 200.66 0)
     (effects (font (size 1.27 1.27)) (justify left bottom))
   )
@@
     (effects (font (size 1.27 1.27)) (justify right bottom))
   )
-  (label "MAIN_A9" (at 142.24 220.98 0)
+  (label "MAIN_AB9" (at 142.24 220.98 0)
     (effects (font (size 1.27 1.27)) (justify left bottom))
   )
@@
     (effects (font (size 1.27 1.27)) (justify left bottom))
   )
-  (label "MAIN_D13" (at 275.59 195.58 0)
+  (label "MAIN_DB13" (at 275.59 195.58 0)
     (effects (font (size 1.27 1.27)) (justify left bottom))
   )
@@
     (effects (font (size 1.27 1.27)) (justify left bottom))
   )
-  (label "MAIN_A10" (at 142.24 238.76 0)
+  (label "MAIN_AB10" (at 142.24 238.76 0)
     (effects (font (size 1.27 1.27)) (justify left bottom))
   )
@@
     (effects (font (size 1.27 1.27)) (justify right bottom))
   )
-  (label "MAIN_D6" (at 276.86 158.75 0)
+  (label "MAIN_DB6" (at 276.86 158.75 0)
     (effects (font (size 1.27 1.27)) (justify left bottom))
   )
@@
     (effects (font (size 1.27 1.27)) (justify right bottom))
   )
-  (label "MAIN_D9" (at 275.59 205.74 0)
+  (label "MAIN_DB9" (at 275.59 205.74 0)
     (effects (font (size 1.27 1.27)) (justify left bottom))
   )
@@
     (effects (font (size 1.27 1.27)) (justify left bottom))
   )
-  (label "MAIN_A3" (at 142.24 228.6 0)
+  (label "MAIN_AB3" (at 142.24 228.6 0)
     (effects (font (size 1.27 1.27)) (justify left bottom))
   )
@@
     (effects (font (size 1.27 1.27)) (justify left bottom))
   )
-  (label "MAIN_D2" (at 276.86 168.91 0)
+  (label "MAIN_DB2" (at 276.86 168.91 0)
     (effects (font (size 1.27 1.27)) (justify left bottom))
   )
@@
     (effects (font (size 1.27 1.27)) (justify left bottom))
   )
-  (label "MAIN_D14" (at 275.59 193.04 0)
+  (label "MAIN_DB14" (at 275.59 193.04 0)
     (effects (font (size 1.27 1.27)) (justify left bottom))
   )
@@
     (effects (font (size 1.27 1.27)) (justify right bottom))
   )
-  (label "MAIN_D8" (at 275.59 208.28 0)
+  (label "MAIN_DB8" (at 275.59 208.28 0)
     (effects (font (size 1.27 1.27)) (justify left bottom))
   )
@@
     (effects (font (size 1.27 1.27)) (justify left bottom))
   )
-  (label "MAIN_A4" (at 142.24 231.14 0)
+  (label "MAIN_AB4" (at 142.24 231.14 0)
     (effects (font (size 1.27 1.27)) (justify left bottom))
   )
@@
     (effects (font (size 1.27 1.27)) (justify right bottom))
   )
-  (label "MAIN_A8" (at 142.24 236.22 0)
+  (label "MAIN_AB8" (at 142.24 236.22 0)
     (effects (font (size 1.27 1.27)) (justify left bottom))
   )
@@
     (effects (font (size 1.27 1.27)) (justify right bottom))
   )
-  (label "MAIN_A7" (at 142.24 223.52 0)
+  (label "MAIN_AB7" (at 142.24 223.52 0)
     (effects (font (size 1.27 1.27)) (justify left bottom))
   )
@@
     (effects (font (size 1.27 1.27)) (justify right bottom))
   )
-  (label "MAIN_D3" (at 276.86 166.37 0)
+  (label "MAIN_DB3" (at 276.86 166.37 0)
     (effects (font (size 1.27 1.27)) (justify left bottom))
   )
@@
     (effects (font (size 1.27 1.27)) (justify left bottom))
   )
-  (label "MAIN_D10" (at 275.59 203.2 0)
+  (label "MAIN_DB10" (at 275.59 203.2 0)
     (effects (font (size 1.27 1.27)) (justify left bottom))
   )
@@
     (effects (font (size 1.27 1.27)) (justify left bottom))
   )
-  (label "MAIN_A6" (at 142.24 233.68 0)
+  (label "MAIN_AB6" (at 142.24 233.68 0)
     (effects (font (size 1.27 1.27)) (justify left bottom))
   )
@@
     (effects (font (size 1.27 1.27)) (justify left bottom))
   )
-  (label "MAIN_D5" (at 276.86 161.29 0)
+  (label "MAIN_DB5" (at 276.86 161.29 0)
     (effects (font (size 1.27 1.27)) (justify left bottom))
   )
@@
     (effects (font (size 1.27 1.27)) (justify left bottom))
   )
-  (label "MAIN_D4" (at 276.86 163.83 0)
+  (label "MAIN_DB4" (at 276.86 163.83 0)
     (effects (font (size 1.27 1.27)) (justify left bottom))
   )
@@
     (effects (font (size 1.27 1.27)) (justify left bottom))
   )
-  (label "MAIN_A5" (at 142.24 226.06 0)
+  (label "MAIN_AB5" (at 142.24 226.06 0)
     (effects (font (size 1.27 1.27)) (justify left bottom))
   )
@@
     (effects (font (size 1.27 1.27)) (justify right bottom))
   )
-  (label "MAIN_D0" (at 276.86 173.99 0)
+  (label "MAIN_DB0" (at 276.86 173.99 0)
     (effects (font (size 1.27 1.27)) (justify left bottom))
   )
@@
     (effects (font (size 1.27 1.27)) (justify right bottom))
   )
-  (label "MAIN_D12" (at 275.59 198.12 0)
+  (label "MAIN_DB12" (at 275.59 198.12 0)
     (effects (font (size 1.27 1.27)) (justify left bottom))
   )
@@
     (effects (font (size 1.27 1.27)) (justify right bottom))
   )
-  (label "MAIN_D1" (at 276.86 171.45 0)
+  (label "MAIN_DB1" (at 276.86 171.45 0)
     (effects (font (size 1.27 1.27)) (justify left bottom))
   )
@@
     (effects (font (size 1.27 1.27)) (justify left bottom))
   )
-  (label "MAIN_D7" (at 276.86 156.21 0)
+  (label "MAIN_DB7" (at 276.86 156.21 0)
     (effects (font (size 1.27 1.27)) (justify left bottom))
   )
@@
     (effects (font (size 1.27 1.27)) (justify right))
   )
-  (hierarchical_label "MAIN_D[0..15]" (shape input) (at 261.62 147.32 180)
+  (hierarchical_label "MAIN_DB[15..0]" (shape input) (at 261.62 147.32 180)
     (effects (font (size 1.27 1.27)) (justify right))
   )
@@
   (symbol (lib_id "power:VCC") (at 339.09 80.01 0) (unit 1)
     (in_bom yes) (on_board yes)
-    (property "Reference" "#PWR0116" (id 0) (at 339.09 83.82 0)
+    (property "Reference" "#PWR?" (id 0) (at 339.09 83.82 0)
       (effects (font (size 1.27 1.27)) hide)
     )
@@
   (symbol (lib_id "power:VSS") (at 266.7 100.33 180) (unit 1)
     (in_bom yes) (on_board yes)
-    (property "Reference" "#PWR0117" (id 0) (at 266.7 96.52 0)
-      (effects (font (size 1.27 1.27)) hide)
-    )
+    (property "Reference" "#PWR?" (id 0) (at 266.7 96.52 0)
+      (effects (font (size 1.27 1.27)) hide)
+    )
