File: cores/s18/sch/gfx_scr.kicad_sch (KiCad schematic)
At the start: 24 parts, among them Q1 74LS244, Q10 74LS367, Q2 74LS244, T10 74LS163, T11 PAL16L8, X4 HM65256B_SERIES, X6 74LS244, Y4 HM65256B_SERIES, Y6 74LS244

Commit message: system 18 schematics transferred after update
Connections:
- net MAIN_A1 is gone; now on net MAIN_AB1: Y6.2 (I0a)
- net MAIN_A10 is gone; now on net MAIN_AB10: X6.13 (I1b)
- net MAIN_A11 is gone; now on net MAIN_AB11: X6.15 (I2b)
- net MAIN_A12 is gone; now on net MAIN_AB12: X6.8 (I3a)
- net MAIN_A13 is gone; now on net MAIN_AB13: X6.6 (I2a)
- net MAIN_A14 is gone; now on net MAIN_AB14: X6.4 (I1a)
- net MAIN_A15 is gone; now on net MAIN_AB15: X6.2 (I0a)
- net MAIN_A2 is gone; now on net MAIN_AB2: Y6.4 (I1a)
- net MAIN_A3 is gone; now on net MAIN_AB3: Y6.6 (I2a)
- net MAIN_A4 is gone; now on net MAIN_AB4: Y6.8 (I3a)
- net MAIN_A5 is gone; now on net MAIN_AB5: Y6.17 (I3b)
- net MAIN_A6 is gone; now on net MAIN_AB6: Y6.15 (I2b)
- net MAIN_A7 is gone; now on net MAIN_AB7: Y6.13 (I1b)
- net MAIN_A8 is gone; now on net MAIN_AB8: Y6.11 (I0b)
- net MAIN_A9 is gone; now on net MAIN_AB9: X6.11 (I0b)
- net ~{CSYNC}: now reaches 4.7kOhms.2, S11.19 (IO1)
- net A10 renamed LATCH10
- net A11 renamed LATCH11
- net A12 renamed LATCH12
- net A13 renamed LATCH13
- net A14 renamed LATCH14
- net A8 renamed LATCH8
- net A9 renamed LATCH9
- net MAIN_A16 renamed MAIN_AB16
- net MAIN_D0 renamed MAIN_DB0
- net MAIN_D1 renamed MAIN_DB1
- net MAIN_D10 renamed MAIN_DB10
- net MAIN_D11 renamed MAIN_DB11
- net MAIN_D12 renamed MAIN_DB12
- net MAIN_D13 renamed MAIN_DB13
- net MAIN_D14 renamed MAIN_DB14
- net MAIN_D15 renamed MAIN_DB15
- net MAIN_D2 renamed MAIN_DB2
- net MAIN_D3 renamed MAIN_DB3
- net MAIN_D4 renamed MAIN_DB4
- net MAIN_D5 renamed MAIN_DB5
- net MAIN_D6 renamed MAIN_DB6
- net MAIN_D7 renamed MAIN_DB7
- net MAIN_D8 renamed MAIN_DB8
- net MAIN_D9 renamed MAIN_DB9
- now unconnected: S11.12 (IO8), S11.13 (IO7), S11.14 (IO6), S11.15 (IO5), S11.16 (IO4), S11.17 (I03), S11.18 (IO2), T11.12 (IO8), T11.13 (IO7), T11.14 (IO6), T11.15 (IO5), T11.16 (IO4), T11.17 (I03), T11.18 (IO2), T11.19 (IO1)
- no-connect marks 39 -> 37
Other:
- note removed: "NOMBRE PARA ESTE BUS"
- moved on the sheet: 4.7kOhms
