File: cores/s18/sch/memorymapper.kicad_sch (KiCad schematic)
At the start: 19 parts, among them CN5 Conn_02x15_Row_Letter_First, M11 Crystal48.000MHz, M6 D8751H-8, P11 MB3771, Q11 74LS74

Commit message: system 18 schematics transferred after update
Connections:
- net MAIN_A1 renamed MAIN_AB1
- net MAIN_A2 renamed MAIN_AB2
- net MAIN_A3 renamed MAIN_AB3
- net MAIN_A4 renamed MAIN_AB4
- net MAIN_A5 renamed MAIN_AB5
Changed lines of the file:
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@@
     (effects (font (size 1.27 1.27)) (justify left bottom))
   )
-  (label "MAIN_A2" (at 351.79 125.73 180)
+  (label "MAIN_AB2" (at 351.79 125.73 180)
     (effects (font (size 1.27 1.27)) (justify right bottom))
   )
@@
     (effects (font (size 1.27 1.27)) (justify right bottom))
   )
-  (label "MAIN_A3" (at 321.31 123.19 0)
+  (label "MAIN_AB3" (at 321.31 123.19 0)
     (effects (font (size 1.27 1.27)) (justify left bottom))
   )
@@
     (effects (font (size 1.27 1.27)) (justify left bottom))
   )
-  (label "MAIN_A4" (at 351.79 123.19 180)
+  (label "MAIN_AB4" (at 351.79 123.19 180)
     (effects (font (size 1.27 1.27)) (justify right bottom))
   )
@@
     (effects (font (size 1.27 1.27)) (justify right bottom))
   )
-  (label "MAIN_A5" (at 321.31 120.65 0)
+  (label "MAIN_AB5" (at 321.31 120.65 0)
     (effects (font (size 1.27 1.27)) (justify left bottom))
   )
@@
     (effects (font (size 1.27 1.27)) (justify right bottom))
   )
-  (label "MAIN_A1" (at 321.31 125.73 0)
+  (label "MAIN_AB1" (at 321.31 125.73 0)
     (effects (font (size 1.27 1.27)) (justify left bottom))
   )
@@
     (effects (font (size 1.27 1.27)) (justify left))
   )
-  (hierarchical_label "ADRESS" (shape input) (at 68.58 147.32 180)
+  (hierarchical_label "MAIN_A[23..1]" (shape input) (at 68.58 147.32 180)
     (effects (font (size 1.27 1.27)) (justify right))
   )
@@
     (effects (font (size 1.27 1.27)) (justify left))
   )
-  (hierarchical_label "DATA" (shape input) (at 52.07 38.1 180)
+  (hierarchical_label "MAIN_D[15..0]" (shape input) (at 52.07 38.1 180)
     (effects (font (size 1.27 1.27)) (justify right))
   )
@@
   (symbol (lib_id "power:VSS") (at 219.71 50.8 180) (unit 1)
     (in_bom yes) (on_board yes)
-    (property "Reference" "#PWR0111" (id 0) (at 219.71 46.99 0)
+    (property "Reference" "#PWR?" (id 0) (at 219.71 46.99 0)
       (effects (font (size 1.27 1.27)) hide)
     )
@@
   (symbol (lib_id "power:VCC") (at 118.11 30.48 0) (unit 1)
     (in_bom yes) (on_board yes)
-    (property "Reference" "#PWR0109" (id 0) (at 118.11 34.29 0)
+    (property "Reference" "#PWR?" (id 0) (at 118.11 34.29 0)
       (effects (font (size 1.27 1.27)) hide)
     )
@@
   (symbol (lib_id "power:VCC") (at 290.83 44.45 0) (unit 1)
     (in_bom yes) (on_board yes)
-    (property "Reference" "#PWR0110" (id 0) (at 290.83 48.26 0)
-      (effects (font (size 1.27 1.27)) hide)
-    )
+    (property "Reference" "#PWR?" (id 0) (at 290.83 48.26 0)
+      (effects (font (size 1.27 1.27)) hide)
+    )
