File: cores/s18/sch/objrom.kicad_sch (KiCad schematic)
At the start: 9 parts

Commit message: system 18 schematics transferred after update
Connections:
- net VDD renamed VCC
Changed lines of the file:
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@@
     (effects (font (size 1.27 1.27)) (justify left bottom))
   )
-  (label "VDD" (at 137.16 43.18 270)
+  (label "VCC" (at 137.16 43.18 270)
     (effects (font (size 1.27 1.27)) (justify right bottom))
   )
@@
     (effects (font (size 1.27 1.27)) (justify left bottom))
   )
-  (label "VDD" (at 334.01 128.27 270)
+  (label "VCC" (at 334.01 128.27 270)
     (effects (font (size 1.27 1.27)) (justify right bottom))
   )
@@
     (effects (font (size 1.27 1.27)) (justify left bottom))
   )
-  (label "VDD" (at 264.16 127 270)
+  (label "VCC" (at 264.16 127 270)
     (effects (font (size 1.27 1.27)) (justify right bottom))
   )
@@
     (effects (font (size 1.27 1.27)) (justify right bottom))
   )
-  (label "VDD" (at 137.16 125.73 270)
+  (label "VCC" (at 137.16 125.73 270)
     (effects (font (size 1.27 1.27)) (justify right bottom))
   )
@@
     (effects (font (size 1.27 1.27)) (justify right bottom))
   )
-  (label "VDD" (at 264.16 44.45 270)
+  (label "VCC" (at 264.16 44.45 270)
     (effects (font (size 1.27 1.27)) (justify right bottom))
   )
@@
     (effects (font (size 1.27 1.27)) (justify left bottom))
   )
-  (label "VDD" (at 334.01 45.72 270)
+  (label "VCC" (at 334.01 45.72 270)
     (effects (font (size 1.27 1.27)) (justify right bottom))
   )
@@
     (effects (font (size 1.27 1.27)) (justify right bottom))
   )
-  (label "VDD" (at 198.12 43.18 270)
+  (label "VCC" (at 198.12 43.18 270)
     (effects (font (size 1.27 1.27)) (justify right bottom))
   )
@@
     (effects (font (size 1.27 1.27)) (justify left bottom))
   )
-  (label "VDD" (at 198.12 125.73 270)
-    (effects (font (size 1.27 1.27)) (justify right bottom))
-  )
+  (label "VCC" (at 198.12 125.73 270)
+    (effects (font (size 1.27 1.27)) (justify right bottom))
+  )
