File: cores/s18/sch/romboard.kicad_sch (KiCad schematic)
At the start: 8 parts, among them CN1 Conn_02x30_Row_Letter_First, CN2 Conn_02x25_Row_Letter_First, CN3 Conn_02x30_Row_Letter_First, CN4 Conn_02x25_Row_Letter_First

Commit message: system 18 schematics transferred after update
Connections:
- net CN4_AB[13..20]: no longer CN4.a20 (Pin_a20)
- net VDD: no longer CN1.a29 (Pin_a29), CN1.a30 (Pin_a30), CN1.b29 (Pin_b29), CN1.b30 (Pin_b30), CN2.a23 (Pin_a23), CN2.a24 (Pin_a24), CN2.a25 (Pin_a25), CN2.b23 (Pin_b23), CN2.b24 (Pin_b24), CN2.b25 (Pin_b25), CN3.a29 (Pin_a29), CN3.a30 (Pin_a30), CN3.b28 (Pin_b28), CN3.b29 (Pin_b29), CN3.b30 (Pin_b30), CN4.a24 (Pin_a24), CN4.a25 (Pin_a25), CN4.b24 (Pin_b24), CN4.b25 (Pin_b25)
- net MAIN_A1 renamed MAIN_AB1
- net MAIN_A10 renamed MAIN_AB10
- net MAIN_A11 renamed MAIN_AB11
- net MAIN_A12 renamed MAIN_AB12
- net MAIN_A13 renamed MAIN_AB13
- net MAIN_A14 renamed MAIN_AB14
- net MAIN_A15 renamed MAIN_AB15
- net MAIN_A16 renamed MAIN_AB16
- net MAIN_A17 renamed MAIN_AB17
- net MAIN_A18 renamed MAIN_AB18
- net MAIN_A2 renamed MAIN_AB2
- net MAIN_A3 renamed MAIN_AB3
- net MAIN_A4 renamed MAIN_AB4
- net MAIN_A5 renamed MAIN_AB5
- net MAIN_A6 renamed MAIN_AB6
- net MAIN_A7 renamed MAIN_AB7
- net MAIN_A8 renamed MAIN_AB8
- net MAIN_A9 renamed MAIN_AB9
- new net CN4_A20: CN4.a20 (Pin_a20)
- new net VCC: CN1.a29 (Pin_a29), CN1.a30 (Pin_a30), CN1.b29 (Pin_b29), CN1.b30 (Pin_b30), CN2.a23 (Pin_a23), CN2.a24 (Pin_a24), CN2.a25 (Pin_a25), CN2.b23 (Pin_b23), CN2.b24 (Pin_b24), CN2.b25 (Pin_b25), CN3.a29 (Pin_a29), CN3.a30 (Pin_a30), CN3.b28 (Pin_b28), CN3.b29 (Pin_b29), CN3.b30 (Pin_b30), CN4.a24 (Pin_a24), CN4.a25 (Pin_a25), CN4.b24 (Pin_b24), CN4.b25 (Pin_b25)
Other:
- sheet cpurom ports: added MAIN_AB[1..18], MAIN_DB[7..0]; removed MAIN_A[1..18], MAIN_D[0..7]
- note removed: "CN1"
- note removed: "CN2"
- note removed: "CN3"
- note removed: "CN4"
- moved on the sheet: C?, CN1, CN2, CN3, CN4
