File: cores/s18/sch/scrrom.kicad_sch (KiCad schematic)
At the start: 7 parts

Commit message: system 18 schematics transferred after update
Connections:
- net VDD renamed VCC
Changed lines of the file:
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@@
     (effects (font (size 1.27 1.27)) (justify left bottom))
   )
-  (label "VDD" (at 299.72 58.42 270)
+  (label "VCC" (at 299.72 58.42 270)
     (effects (font (size 1.27 1.27)) (justify right bottom))
   )
@@
     (effects (font (size 1.27 1.27)) (justify left bottom))
   )
-  (label "VDD" (at 185.42 144.78 180)
+  (label "VCC" (at 185.42 144.78 180)
     (effects (font (size 1.27 1.27)) (justify right bottom))
   )
@@
     (effects (font (size 1.27 1.27)) (justify left bottom))
   )
-  (label "VDD" (at 220.98 118.11 0)
+  (label "VCC" (at 220.98 118.11 0)
     (effects (font (size 1.27 1.27)) (justify left bottom))
   )
@@
     (effects (font (size 1.27 1.27)) (justify left bottom))
   )
-  (label "VDD" (at 240.03 58.42 270)
+  (label "VCC" (at 240.03 58.42 270)
     (effects (font (size 1.27 1.27)) (justify right bottom))
   )
@@
     (effects (font (size 1.27 1.27)) (justify right bottom))
   )
-  (label "VDD" (at 162.56 200.66 0)
+  (label "VCC" (at 162.56 200.66 0)
     (effects (font (size 1.27 1.27)) (justify left bottom))
   )
@@
     (effects (font (size 1.27 1.27)) (justify left bottom))
   )
-  (label "VDD" (at 162.56 118.11 0)
-    (effects (font (size 1.27 1.27)) (justify left bottom))
-  )
-  (label "VDD" (at 238.76 144.78 180)
+  (label "VCC" (at 162.56 118.11 0)
+    (effects (font (size 1.27 1.27)) (justify left bottom))
+  )
+  (label "VCC" (at 238.76 144.78 180)
     (effects (font (size 1.27 1.27)) (justify right bottom))
   )
@@
     (effects (font (size 1.27 1.27)) (justify left bottom))
   )
-  (label "VDD" (at 292.1 144.78 180)
+  (label "VCC" (at 292.1 144.78 180)
     (effects (font (size 1.27 1.27)) (justify right bottom))
   )
@@
     (effects (font (size 1.27 1.27)) (justify right bottom))
   )
-  (label "VDD" (at 280.67 118.11 0)
+  (label "VCC" (at 280.67 118.11 0)
     (effects (font (size 1.27 1.27)) (justify left bottom))
   )
@@
     (effects (font (size 1.27 1.27)) (justify right bottom))
   )
-  (label "VDD" (at 267.97 200.66 0)
+  (label "VCC" (at 267.97 200.66 0)
     (effects (font (size 1.27 1.27)) (justify left bottom))
   )
@@
     (effects (font (size 1.27 1.27)) (justify left bottom))
   )
-  (label "VDD" (at 214.63 200.66 0)
+  (label "VCC" (at 214.63 200.66 0)
     (effects (font (size 1.27 1.27)) (justify left bottom))
   )
@@
     (effects (font (size 1.27 1.27)) (justify left bottom))
   )
-  (label "VDD" (at 181.61 58.42 270)
-    (effects (font (size 1.27 1.27)) (justify right bottom))
-  )
+  (label "VCC" (at 181.61 58.42 270)
+    (effects (font (size 1.27 1.27)) (justify right bottom))
+  )
