File: cores/s18/sch/sound_a.kicad_sch (KiCad schematic)
At the start: 21 parts, among them J3 PAL16L8, K1 ASSP5C68A, K2 74HC245, K4 Z80CPU, M3 74AHC244, Q4 TMM2063AP_10, T4 74LS157, U4 74LS74

Commit message: system 18 schematics transferred after update
Connections:
- net VDD is gone; now on net VCC: J3.20 (VCC), L3.20 (VCC), M3.20 (VCC), Q4.26 (CS2)
- net PAL2: no longer names the net of J3.17 (I03)
- net PAL3: no longer names the net of J3.16 (IO4)
Changed lines of the file:
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@@
   (junction (at 154.94 40.64) (diameter 0) (color 0 0 0 0)
   )
+  (no_connect (at 311.15 130.81))
   (no_connect (at 30.48 248.92))
   (no_connect (at 345.44 220.98))
@@
   (no_connect (at 345.44 223.52))
   (no_connect (at 21.59 223.52))
+  (no_connect (at 311.15 133.35))
   (no_connect (at 208.28 60.96))
   (no_connect (at 165.1 38.1))
@@
   (no_connect (at 26.67 190.5))
   (no_connect (at 30.48 261.62))
-  (no_connect (at 320.04 133.35))
   (no_connect (at 26.67 193.04))
   (no_connect (at 345.44 236.22))
-  (no_connect (at 320.04 130.81))
   (bus_entry (at 274.32 78.74) (size -2.54 2.54)
     (stroke (width 0) (type default) (color 0 0 0 0))
@@
     (stroke (width 0) (type default) (color 0 0 0 0))
   )
-  (wire (pts (xy 311.15 133.35) (xy 320.04 133.35))
-    (stroke (width 0) (type default) (color 0 0 0 0))
-  )
   (wire (pts (xy 64.77 172.72) (xy 80.01 172.72))
     (stroke (width 0) (type default) (color 0 0 0 0))
@@
     (stroke (width 0) (type default) (color 0 0 0 0))
   )
-  (bus (pts (xy 182.88 16.51) (xy 182.88 29.21))
+  (bus (pts (xy 179.07 29.21) (xy 182.88 29.21))
     (stroke (width 0) (type default) (color 0 0 0 0))
   )
@@
     (stroke (width 0) (type default) (color 0 0 0 0))
   )
-  (wire (pts (xy 311.15 130.81) (xy 320.04 130.81))
-    (stroke (width 0) (type default) (color 0 0 0 0))
-  )
   (wire (pts (xy 187.96 116.84) (xy 187.96 125.73))
     (stroke (width 0) (type default) (color 0 0 0 0))
@@
     (effects (font (size 1.27 1.27)) (justify left bottom))
   )
-  (label "VDD" (at 276.86 99.06 0)
+  (label "VCC" (at 276.86 99.06 0)
     (effects (font (size 1.27 1.27)) (justify left bottom))
   )
@@
     (effects (font (size 1.27 1.27)) (justify right bottom))
   )
-  (label "VDD" (at 245.11 116.84 0)
+  (label "VCC" (at 245.11 116.84 0)
     (effects (font (size 1.27 1.27)) (justify left bottom))
   )
@@
     (effects (font (size 1.27 1.27)) (justify left bottom))
   )
-  (label "PAL2" (at 320.04 130.81 180)
-    (effects (font (size 1.27 1.27)) (justify right bottom))
-  )
   (label "AB0" (at 166.37 200.66 0)
     (effects (font (size 1.27 1.27)) (justify left bottom))
@@
     (effects (font (size 1.27 1.27)) (justify left bottom))
   )
-  (label "PAL3" (at 320.04 133.35 180)
-    (effects (font (size 1.27 1.27)) (justify right bottom))
-  )
   (label "A7" (at 68.58 180.34 0)
     (effects (font (size 1.27 1.27)) (justify left bottom))
@@
     (effects (font (size 1.27 1.27)) (justify right bottom))
   )
-  (label "VDD" (at 298.45 116.84 0)
+  (label "VCC" (at 298.45 116.84 0)
     (effects (font (size 1.27 1.27)) (justify left bottom))
   )
@@
     (effects (font (size 1.27 1.27)) (justify right bottom))
   )
-  (label "VDD" (at 246.38 59.69 0)
+  (label "VCC" (at 246.38 59.69 0)
     (effects (font (size 1.27 1.27)) (justify left bottom))
   )
@@
     (effects (font (size 1.27 1.27)) (justify left))
   )
-  (hierarchical_label "SND_D[0..7]" (shape bidirectional) (at 182.88 16.51 180)
+  (hierarchical_label "SND_D[0..7]" (shape bidirectional) (at 179.07 29.21 180)
     (effects (font (size 1.27 1.27)) (justify right))
   )
@@
   (symbol (lib_id "power:VCC") (at 156.21 19.05 0) (mirror y) (unit 1)
     (in_bom yes) (on_board yes)
-    (property "Reference" "#PWR0120" (id 0) (at 156.21 22.86 0)
+    (property "Reference" "#PWR?" (id 0) (at 156.21 22.86 0)
       (effects (font (size 1.27 1.27)) hide)
     )
@@
   (symbol (lib_id "power:VSS") (at 128.27 22.86 180) (unit 1)
     (in_bom yes) (on_board yes)
-    (property "Reference" "#PWR0121" (id 0) (at 128.27 19.05 0)
+    (property "Reference" "#PWR?" (id 0) (at 128.27 19.05 0)
       (effects (font (size 1.27 1.27)) hide)
     )
@@
   (symbol (lib_id "power:VCC") (at 46.99 151.13 0) (unit 1)
     (in_bom yes) (on_board yes)
-    (property "Reference" "#PWR0123" (id 0) (at 46.99 154.94 0)
+    (property "Reference" "#PWR?" (id 0) (at 46.99 154.94 0)
       (effects (font (size 1.27 1.27)) hide)
     )
@@
   (symbol (lib_id "power:VSS") (at 46.99 236.22 180) (unit 1)
     (in_bom yes) (on_board yes)
-    (property "Reference" "#PWR0122" (id 0) (at 46.99 232.41 0)
+    (property "Reference" "#PWR?" (id 0) (at 46.99 232.41 0)
       (effects (font (size 1.27 1.27)) hide)
     )
