File: cores/s18/sch/system18.kicad_sch (KiCad schematic)
At the start: 1 part

Commit message: system 18 schematics transferred after update
Connections:
- net VCAB is gone; now on net VCC: JM1.4 (+5V)
- net VIDEO_GND is gone; now on net VSS: JM1.14 (VIDEO_GND)
- net VSS: no longer JM1.5 (-5V), JM1.E (-5V)
- net UK_SND renamed N.C
- net VCCA12v renamed +12V
- new net -5V: JM1.5 (-5V), JM1.E (-5V)
Other:
- sheet colmix ports: added COLA[10..0], MAIN_AB[11..1], MAIN_DB[15..0]; removed A[0..10], COLMIX, MAIN_A[1..23], MAIN_D[0..15]
- sheet gfx_main ports: added B_ANLONG, CN1_A24, EDCK, G_ANLONG, MAIN_AB[23..1], MAIN_DB[15..0], MCK, R_ANLONG, SPA_B, ~{CSYNC}, ~{RESET}, ~{VSYNC}; removed MAIN_A[1..23], MAIN_D[0..15]
- sheet gfx_obj ports: added MAIN_AB[1..18], MAIN_DB[15..0]; removed MAIN_A[1..18], MAIN_D[0..15]
- sheet gfx_scr ports: added COLA[10..0], MAIN_DB[15..0]; removed COLA[0..10], MAIN_D[0..15]
- sheet main ports: added MAIN_AB[23..1], MAIN_A[23..1], MAIN_DB[15..0], MAIN_D[15..0]; removed ADRESS, DATA, MAIN_A[1..23], MAIN_D[0..15]
- sheet memorymapper ports: added MAIN_A[23..1], MAIN_D[15..0]; removed ADRESS, DATA
- sheet romboard ports: added MAIN_AB[1..18], MAIN_DB[7..0]; removed MAIN_A[1..18], MAIN_D[0..7]
- note added: "*"
- note removed: "OK"
- note removed: "ok"
